File: Hardware/Christmas_Kit.brd (EAGLE design)
At the start: 105.4 x 116 mm, 17 parts, among them U2 ATTINY13DIP, U4 AVR_SPI_PRG_6PTH

Commit message: Updated revision to symbol
Parts:
- added U$1: REVISION, SparkFun-Aesthetics:REVISION
Other:
- board text added: "R. Owens"
- board text added: "T. Klopfenstein"
- board text removed: "R. Owens, Revision by: T. Klopfenstein"
